Commit message: control gripper and manipulator_p with moveit2 updated

File: mani_p_description/robot/mani_p.core.xacro (robot description, xacro)
@@ -27,19 +27,19 @@
       <geometry>
         <mesh
-          filename="file://$(find mani_p_description)/meshes/Base_link.STL" />
-      </geometry>
-      <material
-        name="">
-        <color
-          rgba="0.792156862745098 0.819607843137255 0.933333333333333 1" />
-      </material>
-    </visual>
-    <collision>
-      <origin
-        xyz="0 0 0"
-        rpy="0 0 0" />
-      <geometry>
-        <mesh
-          filename="file://$(find mani_p_description)/meshes/Base_link.STL" />
+          filename="file://$(find mani_p_description)/meshes/table_visual.STL" />
+      </geometry>
+      <material
+        name="">
+        <color
+          rgba="0.792156862745098 0.819607843137255 0.933333333333333 1" />
+      </material>
+    </visual>
+    <collision>
+      <origin
+        xyz="0 0 0"
+        rpy="0 0 0" />
+      <geometry>
+        <mesh
+          filename="file://$(find mani_p_description)/meshes/table_collision.STL" />
       </geometry>
     </collision>
@@ -67,5 +67,5 @@
       <geometry>
         <mesh
-          filename="file://$(find mani_p_description)/meshes/Base_arm.STL" />
+          filename="file://$(find mani_p_description)/meshes/Base_arm_visual.stl" />
       </geometry>
       <material
@@ -81,5 +81,5 @@
       <geometry>
         <mesh
-          filename="file://$(find mani_p_description)/meshes/Base_arm.STL" />
+          filename="file://$(find mani_p_description)/meshes/base_collision.STL" />
       </geometry>
     </collision>
@@ -87,7 +87,7 @@
   <joint
     name="Base_arm_J0"
-    type="prismatic">
-    <origin
-      xyz="0 0 -0.0286185637769465"
+    type="fixed">
+    <origin
+      xyz="0 0 0.04"
       rpy="0 0 0" />
     <parent
@@ -125,5 +125,5 @@
       <geometry>
         <mesh
-          filename="file://$(find mani_p_description)/meshes/L1.STL" />
+          filename="file://$(find mani_p_description)/meshes/L1_visual.stl" />
       </geometry>
       <material
@@ -183,5 +183,5 @@
       <geometry>
         <mesh
-          filename="file://$(find mani_p_description)/meshes/L2.STL" />
+          filename="file://$(find mani_p_description)/meshes/L2_visual.stl" />
       </geometry>
       <material
@@ -215,5 +215,5 @@
     <limit
       lower="-1.57"
-      upper="0"
+      upper="1.57"
       effort="200"
       velocity="3" />
@@ -241,20 +241,20 @@
       <geometry>
         <mesh
+          filename="file://$(find mani_p_description)/meshes/L3_visual.stl" />
+      </geometry>
+      <material
+        name="">
+        <color
+          rgba="0.792156862745098 0.819607843137255 0.933333333333333 1" />
+      </material>
+    </visual>
+    <collision>
+      <origin
+        xyz="0 0 0"
+        rpy="0 0 0" />
+      <geometry>
+        <mesh
           filename="file://$(find mani_p_description)/meshes/L3.STL" />
       </geometry>
-      <material
-        name="">
-        <color
-          rgba="0.792156862745098 0.819607843137255 0.933333333333333 1" />
-      </material>
-    </visual>
-    <collision>
-      <origin
-        xyz="0 0 0"
-        rpy="0 0 0" />
-      <geometry>
-        <mesh
-          filename="file://$(find mani_p_description)/meshes/L3.STL" />
-      </geometry>
     </collision>
   </link>
@@ -264,5 +264,5 @@
     <origin
       xyz="0.264000000000014 0.0299999999999664 0"
-      rpy="0 0 0" />
+      rpy="0 0 0.7854" />
     <parent
       link="L2" />
@@ -272,6 +272,6 @@
       xyz="0 0 -1" />
     <limit
-      lower="-1.57"
-      upper="0"
+      lower="-2.3562"
+      upper="1.57"
       effort="200"
       velocity="3" />
@@ -299,5 +299,5 @@
       <geometry>
         <mesh
-          filename="file://$(find mani_p_description)/meshes/L4.STL" />
+          filename="file://$(find mani_p_description)/meshes/L4_visual.stl" />
       </geometry>
       <material
@@ -357,5 +357,5 @@
       <geometry>
         <mesh
-          filename="file://$(find mani_p_description)/meshes/L5.STL" />
+          filename="file://$(find mani_p_description)/meshes/L5_visual.stl" />
       </geometry>
       <material
@@ -389,5 +389,5 @@
     <limit
       lower="-1.57"
-      upper="0"
+      upper="1.57"
       effort="200"
       velocity="3" />
@@ -415,19 +415,19 @@
       <geometry>
         <mesh
-          filename="file://$(find mani_p_description)/meshes/Gripper.STL" />
-      </geometry>
-      <material
-        name="">
-        <color
-          rgba="0.792156862745098 0.819607843137255 0.933333333333333 1" />
-      </material>
-    </visual>
-    <collision>
-      <origin
-        xyz="0 0 0"
-        rpy="0 0 0" />
-      <geometry>
-        <mesh
-          filename="file://$(find mani_p_description)/meshes/Gripper.STL" />
+          filename="file://$(find mani_p_description)/meshes/Gripper_visual.stl" />
+      </geometry>
+      <material
+        name="">
+        <color
+          rgba="0.792156862745098 0.819607843137255 0.933333333333333 1" />
+      </material>
+    </visual>
+    <collision>
+      <origin
+        xyz="0 0 0"
+        rpy="0 0 0" />
+      <geometry>
+        <mesh
+          filename="file://$(find mani_p_description)/meshes/Gripper_collision.STL" />
       </geometry>
     </collision>

File: mani_p_description/robot/mani_p.ros2.control.xacro (robot description, xacro)
@@ -22,7 +22,15 @@
         <joint name="J3">
             <param name="id">3</param>
-            <command_interface name="position"/>
-            <state_interface name="position"/>
-            <state_interface name="velocity"/>
+            <command_interface name="position">
+                <param name="multiplier">-1</param>
+                <param name="offset">2.356</param>
+            </command_interface>
+            <state_interface name="position">
+              <param name="multiplier">-1</param>
+              <param name="offset">2.356</param>
+            </state_interface>
+            <state_interface name="velocity">
+                <param name="multiplier">-1</param>
+            </state_interface>
         </joint>
         <joint name="J4">

File: mani_p_moveit_config/config/Manipulator_station_urdf_2.ros2_control.xacro (robot description, xacro)
@@ -23,9 +23,16 @@
             </joint>
             <joint name="J3">
-                <command_interface name="position"/>
+                <command_interface name="position">
+                    <param name="multiplier">-1</param>
+                    <param name="offset">2.356</param>
+                </command_interface>
                 <state_interface name="position">
                   <param name="initial_value">${initial_positions['J3']}</param>
+                  <param name="multiplier">-1</param>
+                  <param name="offset">2.356</param>
                 </state_interface>
-                <state_interface name="velocity"/>
+                <state_interface name="velocity">
+                    <param name="multiplier">-1</param>
+                </state_interface>
             </joint>
             <joint name="J4">
