Commit message: moveit2 collision shelf updated

File: mani_p_description/robot/mani_p.sensors.xacro (robot description, xacro)
@@ -21,5 +21,5 @@
         <parent link="$(arg camera_name)_camera_link"/> <!-- Ensure Base_linkis defined in the included files -->
         <child link="Base_link"/> <!-- Ensure zed_camera_link is defined in the ZED macro -->
-        <origin xyz="0.265 0 -0.85" rpy="0 0 0"/>
+        <origin xyz="0.235 0 -0.88" rpy="0 0 0"/>
       </joint>
     </xacro:if>
@@ -29,5 +29,5 @@
         <parent link="Base_link"/>
         <child link="$(arg camera_name)_camera_link"/>
-        <origin xyz="-0.075 0 0.75" rpy="0 0 0"/>
+        <origin xyz="-0.105 0 0.78" rpy="0 0 0"/>
       </joint>
     </xacro:unless>

Commit message: C2F test update

File: mani_p_description/robot/mani_p.sensors.xacro (robot description, xacro)
@@ -34,5 +34,5 @@
     <xacro:include filename="$(find realsense2_description)/urdf/_d435i.urdf.xacro"/>
     <xacro:sensor_d435i parent="palm_link" name="d435i_camera">
-      <origin xyz="0.1 0 0.1" rpy="0 -1.57 0"/>
+      <origin xyz="0.15 0 0.055" rpy="0 -1.57 0"/>
     </xacro:sensor_d435i>
 </robot>

Commit message: fisheye_came tf updated

File: mani_p_description/robot/mani_p.sensors.xacro (robot description, xacro)
@@ -32,7 +32,25 @@
       </joint>
     </xacro:unless>
-    <xacro:include filename="$(find realsense2_description)/urdf/_d435i.urdf.xacro"/>
-    <xacro:sensor_d435i parent="palm_link" name="d435i_camera">
+    <!-- Fisheye Camera Macro -->
+    <xacro:macro name="sensor_fisheye" params="parent name *origin">
+      <joint name="${name}_joint" type="fixed">
+        <xacro:insert_block name="origin" />
+        <parent link="${parent}"/>
+        <child link="${name}_link"/>
+      </joint>
+      <link name="${name}_link">
+        <visual>
+          <geometry>
+            <box size="0.03 0.03 0.03"/>
+          </geometry>
+          <material name="black">
+            <color rgba="0 0 0 1"/>
+          </material>
+        </visual>
+      </link>
+    </xacro:macro>
+    <!-- Fisheye Camera Instance -->
+    <xacro:sensor_fisheye parent="palm_link" name="fisheye_camera">
       <origin xyz="0.15 0 0.055" rpy="0 -1.57 0"/>
-    </xacro:sensor_d435i>
+    </xacro:sensor_fisheye>
 </robot>

Commit message: d345 launch remove

File: mani_p_description/robot/mani_p.sensors.xacro (robot description, xacro)
@@ -52,5 +52,5 @@
     <!-- Fisheye Camera Instance -->
     <xacro:sensor_fisheye parent="palm_link" name="fisheye_camera">
-      <origin xyz="0.15 0 0.055" rpy="0 -1.57 0"/>
+      <origin xyz="0.13 0 0.04" rpy="0 -1.57 0"/>
     </xacro:sensor_fisheye>
 </robot>

Commit message: update shelf1

File: mani_p_description/robot/mani_p.sensors.xacro (robot description, xacro)
@@ -52,5 +52,5 @@
     <!-- Fisheye Camera Instance -->
     <xacro:sensor_fisheye parent="palm_link" name="fisheye_camera">
-      <origin xyz="0.13 0 0.04" rpy="0 -1.57 0"/>
+      <origin xyz="0.075 0 0.12" rpy="0 0 1.57"/>
     </xacro:sensor_fisheye>
 </robot>

Commit message: cube leveler

File: mani_p_description/robot/mani_p.sensors.xacro (robot description, xacro)
@@ -29,5 +29,5 @@
         <parent link="Base_link"/>
         <child link="$(arg camera_name)_camera_link"/>
-        <origin xyz="-0.105 0 0.78" rpy="0 0 0"/>
+        <origin xyz="-0.105 0 0.73" rpy="0 0 0"/>
       </joint>
     </xacro:unless>

Commit message: parameter update

File: mani_p_description/robot/mani_p.sensors.xacro (robot description, xacro)
@@ -29,5 +29,5 @@
         <parent link="Base_link"/>
         <child link="$(arg camera_name)_camera_link"/>
-        <origin xyz="-0.105 0 0.73" rpy="0 0 0"/>
+        <origin xyz="-0.105 0 0.78" rpy="0 0 0"/>
       </joint>
     </xacro:unless>
