Commit message: manipulator controlling updated

File: mani_p_description/robot/mani_p.core2.xacro (robot description, xacro)
@@ -749,3 +749,24 @@
     <limit lower="-0.84901" upper="0.45099" effort="10.0" velocity="1.0" />
   </joint>
+  <link name="tcp_link">
+    <inertial>
+      <origin xyz="0 0 0" rpy="0 0 0" />
+      <mass value="0.001" />
+      <inertia ixx="0.000001" ixy="0" ixz="0" iyy="0.000001" iyz="0" izz="0.000001" />
+    </inertial>
+    <visual>
+      <origin xyz="0 0 0" rpy="0 0 0" />
+      <geometry>
+        <box size="0.02 0.02 0.02" />
+      </geometry>
+      <material name="red">
+        <color rgba="1 0 0 1" />
+      </material>
+    </visual>
+  </link>
+  <joint name="tcp_joint" type="fixed">
+    <origin xyz="0 0 0.25" rpy="0 0 0" />
+    <parent link="palm_link" />
+    <child link="tcp_link" />
+  </joint>
 </robot>

Commit message: action_sever_code updated

File: mani_p_description/robot/mani_p.core2.xacro (robot description, xacro)
@@ -747,5 +747,5 @@
     <axis
       xyz="0 0 -1" />
-    <limit lower="-0.84901" upper="0.45099" effort="10.0" velocity="1.0" />
+    <limit lower="-1.2" upper="0.45099" effort="10.0" velocity="1.0" />
   </joint>
   <link name="tcp_link">

Commit message: commeent updated

File: mani_p_description/robot/mani_p.core2.xacro (robot description, xacro)
@@ -747,5 +747,5 @@
     <axis
       xyz="0 0 -1" />
-    <limit lower="-1.2" upper="0.45099" effort="10.0" velocity="1.0" />
+    <limit lower="-1.57" upper="0.45099" effort="10.0" velocity="1.0" />
   </joint>
   <link name="tcp_link">

Commit message: parameter adjust

File: mani_p_description/robot/mani_p.core2.xacro (robot description, xacro)
@@ -766,5 +766,5 @@
   </link>
   <joint name="tcp_joint" type="fixed">
-    <origin xyz="0 0 0.25" rpy="0 0 0" />
+    <origin xyz="0 0 0.335" rpy="0 0 0" />
     <parent link="palm_link" />
     <child link="tcp_link" />
